File: kicad/billboard/billboard.kicad_sch (KiCad schematic)
At the start: 11 parts

Commit message: Panout 현상 fix
Parts:
- added R? (x2): 1K, symbol Device:R
- added R?: 10K, symbol Device:R
Connections:
- net +5V: now also R?.1, R?.1
- net CK: now also R?.2
- net CS: now also R?.1
- net DO: now also R?.2
- net Earth: now also R?.2
Changed lines of the file:
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@@
 (kicad_sch (version 20211123) (generator eeschema)
   (paper "A4")
+  (junction (at 185.42 86.36) (diameter 0) (color 0 0 0 0)
+  )
   (junction (at 184.15 129.54) (diameter 0) (color 0 0 0 0)
   )
@@
     (stroke (width 0) (type default) (color 0 0 0 0))
   )
+  (wire (pts (xy 180.34 96.52) (xy 180.34 104.14))
+    (stroke (width 0) (type default) (color 0 0 0 0))
+  )
   (wire (pts (xy 99.06 114.3) (xy 111.76 114.3))
     (stroke (width 0) (type default) (color 0 0 0 0))
@@
     (stroke (width 0) (type default) (color 0 0 0 0))
   )
+  (wire (pts (xy 189.23 101.6) (xy 189.23 96.52))
+    (stroke (width 0) (type default) (color 0 0 0 0))
+  )
   (wire (pts (xy 127 88.9) (xy 127 92.71))
     (stroke (width 0) (type default) (color 0 0 0 0))
@@
     (stroke (width 0) (type default) (color 0 0 0 0))
   )
+  (wire (pts (xy 185.42 86.36) (xy 189.23 86.36))
+    (stroke (width 0) (type default) (color 0 0 0 0))
+  )
   (wire (pts (xy 165.1 64.77) (xy 165.1 67.31))
     (stroke (width 0) (type default) (color 0 0 0 0))
@@
     (stroke (width 0) (type default) (color 0 0 0 0))
   )
+  (wire (pts (xy 185.42 85.09) (xy 185.42 86.36))
+    (stroke (width 0) (type default) (color 0 0 0 0))
+  )
   (wire (pts (xy 96.52 64.77) (xy 104.14 64.77))
     (stroke (width 0) (type default) (color 0 0 0 0))
@@
     (stroke (width 0) (type default) (color 0 0 0 0))
   )
+  (wire (pts (xy 200.66 85.09) (xy 200.66 87.63))
+    (stroke (width 0) (type default) (color 0 0 0 0))
+  )
+  (wire (pts (xy 180.34 88.9) (xy 180.34 86.36))
+    (stroke (width 0) (type default) (color 0 0 0 0))
+  )
   (wire (pts (xy 91.44 86.36) (xy 91.44 91.44))
     (stroke (width 0) (type default) (color 0 0 0 0))
@@
     (stroke (width 0) (type default) (color 0 0 0 0))
   )
+  (wire (pts (xy 180.34 86.36) (xy 185.42 86.36))
+    (stroke (width 0) (type default) (color 0 0 0 0))
+  )
   (wire (pts (xy 210.82 119.38) (xy 227.33 119.38))
     (stroke (width 0) (type default) (color 0 0 0 0))
@@
     (stroke (width 0) (type default) (color 0 0 0 0))
   )
-  (wire (pts (xy 213.36 101.6) (xy 203.2 101.6))
+  (wire (pts (xy 189.23 101.6) (xy 213.36 101.6))
     (stroke (width 0) (type default) (color 0 0 0 0))
   )
@@
     (stroke (width 0) (type default) (color 0 0 0 0))
   )
+  (wire (pts (xy 189.23 86.36) (xy 189.23 88.9))
+    (stroke (width 0) (type default) (color 0 0 0 0))
+  )
   (wire (pts (xy 116.84 119.38) (xy 116.84 116.84))
     (stroke (width 0) (type default) (color 0 0 0 0))
@@
     (stroke (width 0) (type default) (color 0 0 0 0))
   )
-  (wire (pts (xy 213.36 77.47) (xy 203.2 77.47))
+  (wire (pts (xy 200.66 77.47) (xy 213.36 77.47))
     (stroke (width 0) (type default) (color 0 0 0 0))
   )
@@
     (stroke (width 0) (type default) (color 0 0 0 0))
   )
-  (wire (pts (xy 213.36 104.14) (xy 203.2 104.14))
+  (wire (pts (xy 180.34 104.14) (xy 213.36 104.14))
     (stroke (width 0) (type default) (color 0 0 0 0))
   )
@@
     (effects (font (size 1.27 1.27)) (justify left bottom))
   )
+  (symbol (lib_id "power:+5V") (at 185.42 85.09 0) (unit 1)
+    (in_bom yes) (on_board yes) (fields_autoplaced)
+    (property "Reference" "#PWR?" (id 0) (at 185.42 88.9 0)
+      (effects (font (size 1.27 1.27)) hide)
+    )
+    (property "Value" "+5V" (id 1) (at 185.42 80.01 0))
+    (property "Footprint" "" (id 2) (at 185.42 85.09 0)
+      (effects (font (size 1.27 1.27)) hide)
+    )
+    (property "Datasheet" "" (id 3) (at 185.42 85.09 0)
+      (effects (font (size 1.27 1.27)) hide)
+    )
+    (pin "1")
+  )
   (symbol (lib_id "power:Earth") (at 111.76 135.89 0) (unit 1)
     (in_bom yes) (on_board yes) (fields_autoplaced)
@@
     )
     (pin "1")
+  )
+  (symbol (lib_id "Device:R") (at 189.23 92.71 0) (unit 1)
+    (in_bom yes) (on_board yes) (fields_autoplaced)
+    (property "Reference" "R?" (id 0) (at 191.77 91.4399 0)
+      (effects (font (size 1.27 1.27)) (justify left))
+    )
+    (property "Value" "1K" (id 1) (at 191.77 93.9799 0)
+      (effects (font (size 1.27 1.27)) (justify left))
+    )
+    (property "Footprint" "" (id 2) (at 187.452 92.71 90)
+      (effects (font (size 1.27 1.27)) hide)
+    )
+    (property "Datasheet" "~" (id 3) (at 189.23 92.71 0)
+      (effects (font (size 1.27 1.27)) hide)
+    )
+    (pin "1")
+    (pin "2")
   )
   (symbol (lib_id "power:Earth") (at 227.33 123.19 0) (unit 1)
@@
     (pin "2")
   )
+  (symbol (lib_id "power:Earth") (at 200.66 87.63 0) (unit 1)
+    (in_bom yes) (on_board yes) (fields_autoplaced)
+    (property "Reference" "#PWR?" (id 0) (at 200.66 93.98 0)
+      (effects (font (size 1.27 1.27)) hide)
+    )
+    (property "Value" "Earth" (id 1) (at 200.66 91.44 0)
+      (effects (font (size 1.27 1.27)) hide)
+    )
+    (property "Footprint" "" (id 2) (at 200.66 87.63 0)
+      (effects (font (size 1.27 1.27)) hide)
+    )
+    (property "Datasheet" "~" (id 3) (at 200.66 87.63 0)
+      (effects (font (size 1.27 1.27)) hide)
+    )
+    (pin "1")
+  )
+  (symbol (lib_id "Device:R") (at 180.34 92.71 0) (unit 1)
+    (in_bom yes) (on_board yes) (fields_autoplaced)
+    (property "Reference" "R?" (id 0) (at 182.88 91.4399 0)
+      (effects (font (size 1.27 1.27)) (justify left))
+    )
+    (property "Value" "1K" (id 1) (at 182.88 93.9799 0)
+      (effects (font (size 1.27 1.27)) (justify left))
+    )
+    (property "Footprint" "" (id 2) (at 178.562 92.71 90)
+      (effects (font (size 1.27 1.27)) hide)
+    )
+    (property "Datasheet" "~" (id 3) (at 180.34 92.71 0)
+      (effects (font (size 1.27 1.27)) hide)
+    )
+    (pin "1")
+    (pin "2")
+  )
   (symbol (lib_id "power:Earth") (at 114.3 67.31 0) (unit 1)
     (in_bom yes) (on_board yes) (fields_autoplaced)
@@
     (pin "2")
   )
+  (symbol (lib_id "Device:R") (at 200.66 81.28 0) (unit 1)
+    (in_bom yes) (on_board yes) (fields_autoplaced)
+    (property "Reference" "R?" (id 0) (at 203.2 80.0099 0)
+      (effects (font (size 1.27 1.27)) (justify left))
+    )
+    (property "Value" "10K" (id 1) (at 203.2 82.5499 0)
+      (effects (font (size 1.27 1.27)) (justify left))
+    )
+    (property "Footprint" "" (id 2) (at 198.882 81.28 90)
+      (effects (font (size 1.27 1.27)) hide)
+    )
+    (property "Datasheet" "~" (id 3) (at 200.66 81.28 0)
+      (effects (font (size 1.27 1.27)) hide)
+    )
+    (pin "1")
+    (pin "2")
+  )
   (symbol (lib_id "power:+3.3V") (at 91.44 86.36 0) (unit 1)
     (in_bom yes) (on_board yes) (fields_autoplaced)
@@
   )
   (symbol_instances
+    (path "/04ad3b31-d796-4075-8823-6b3d286fd40e"
+      (reference "#PWR?") (unit 1) (value "+5V") (footprint "")
+    )
     (path "/1577cdbc-0b6a-4b78-b391-ef6027d98d9a"
       (reference "#PWR?") (unit 1) (value "Earth") (footprint "")
@@
       (reference "#PWR?") (unit 1) (value "+3.3V") (footprint "")
     )
+    (path "/5eb66693-ab1b-4459-a77e-81bcb06ca4d6"
+      (reference "#PWR?") (unit 1) (value "Earth") (footprint "")
+    )
     (path "/697b8b5a-7575-4714-a980-90fdb6cefa55"
       (reference "#PWR?") (unit 1) (value "Earth") (footprint "")
@@
       (reference "JP?") (unit 1) (value "Jumper_2_Open") (footprint "")
     )
+    (path "/18648368-8315-41f6-b287-55706b48f79e"
+      (reference "R?") (unit 1) (value "1K") (footprint "")
+    )
     (path "/3ad6a5dc-b356-4b75-b6fa-f65c46e73e27"
       (reference "R?") (unit 1) (value "1K") (footprint "")
     )
+    (path "/6916b03b-1110-449f-9f3c-ab347cf003e7"
+      (reference "R?") (unit 1) (value "1K") (footprint "")
+    )
+    (path "/a65cad0c-0ef1-4ea5-a965-4eae7ac1f6af"
+      (reference "R?") (unit 1) (value "10K") (footprint "")
+    )
     (path "/47aec22b-82e9-4b91-989d-e048280cce6f"
